File: QSFP_Breakout.kicad_pcb (KiCad board)
At the start: 4 copper layers, 70 x 47.5 mm, 54 parts, among them J1 PCIe_6Pin, J10 RX4_P, J11 TX1_N, J12 TX1_P, J13 TX2_N, J14 TX2_P, J15 TX3_N, J16 TX3_P, J17 TX4_N, J18 TX4_P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

Commit message: Updated GND Fill
Routing:
- net GND: track 910.6 -> 962.1 mm, vias 230 -> 234
- net +3V3: track 168.2 -> 166.4 mm
